File: sch/NMEA_BatteryMonitor 1-2.sch (EAGLE design)
At the start: 9 parts, among them IC1 5V, IC2 INA226, IC3 MCP2562, X3 DS1820

Commit message: initial version
Parts:
- added X2: (no value), con-ptr500:AK500/5
Connections:
- new net N$5: D1.A, X2-1.KL
- new net N$9: IC2.IN+, R2.2, X1-2.KL
- net 12V: no longer D1.A
- net CANH: now also X2-4.KL; no longer X1-5.KL
- net CANL: now also X2-3.KL; no longer X1-4.KL
- net GND: now also X2-2.KL; no longer IC2.IN+, R2.2, X1-2.KL
Other:
- note added: "A"
- note added: "Supply voltage for ESP32 from NEMA Bus"
Changed lines of the file:
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@@
 <part name="D1" library="diode" library_urn="urn:adsk.eagle:library:210" deviceset="1N4004" device="" package3d_urn="urn:adsk.eagle:package:43336/1" value="1N4001"/>
 <part name="X1" library="con-ptr500" library_urn="urn:adsk.eagle:library:181" deviceset="AK500/5" device="" package3d_urn="urn:adsk.eagle:package:9890/1"/>
+<part name="X2" library="con-ptr500" library_urn="urn:adsk.eagle:library:181" deviceset="AK500/5" device="" package3d_urn="urn:adsk.eagle:package:9890/1"/>
 </parts>
 <sheets>
@@
 <text x="2.54" y="132.08" size="1.778" layer="97">To Load</text>
 <text x="2.54" y="160.02" size="1.778" layer="97">Battery +</text>
+<text x="165.1" y="33.02" size="1.778" layer="97">Supply voltage for ESP32 from NEMA Bus</text>
+<text x="255.016" y="5.842" size="5.08" layer="97">A</text>
 </plain>
 <instances>
@@
 <attribute name="NAME" x="19.05" y="130.429" size="1.778" layer="95" rot="R180"/>
 </instance>
-<instance part="X1" gate="-4" x="27.94" y="53.34" smashed="yes">
+<instance part="X2" gate="-1" x="25.4" y="93.98" smashed="yes">
+<attribute name="NAME" x="24.13" y="94.869" size="1.778" layer="95" rot="R180"/>
+</instance>
+<instance part="X2" gate="-2" x="25.4" y="76.2" smashed="yes">
+<attribute name="NAME" x="24.13" y="77.089" size="1.778" layer="95" rot="R180"/>
+</instance>
+<instance part="X2" gate="-3" x="27.94" y="53.34" smashed="yes">
 <attribute name="NAME" x="26.67" y="54.229" size="1.778" layer="95" rot="R180"/>
 </instance>
-<instance part="X1" gate="-5" x="27.94" y="48.26" smashed="yes">
+<instance part="X2" gate="-4" x="27.94" y="48.26" smashed="yes">
 <attribute name="NAME" x="26.67" y="49.149" size="1.778" layer="95" rot="R180"/>
-<attribute name="VALUE" x="24.13" y="44.577" size="1.778" layer="96"/>
 </instance>
 </instances>
@@
 <wire x1="60.96" y1="76.2" x2="60.96" y2="48.26" width="0.1524" layer="91"/>
 <junction x="60.96" y="76.2"/>
-<wire x1="144.78" y1="76.2" x2="144.78" y2="152.4" width="0.1524" layer="91"/>
+<wire x1="144.78" y1="76.2" x2="144.78" y2="144.78" width="0.1524" layer="91"/>
 <pinref part="X3" gate="-3" pin="S"/>
+<wire x1="144.78" y1="144.78" x2="144.78" y2="152.4" width="0.1524" layer="91"/>
 <wire x1="233.68" y1="139.7" x2="233.68" y2="152.4" width="0.1524" layer="91"/>
 <wire x1="233.68" y1="152.4" x2="233.68" y2="160.02" width="0.1524" layer="91"/>
@@
 <pinref part="IC2" gate="G$1" pin="GND"/>
 <wire x1="83.82" y1="149.86" x2="83.82" y2="144.78" width="0.1524" layer="91"/>
-<pinref part="IC2" gate="G$1" pin="IN+"/>
-<wire x1="68.58" y1="149.86" x2="68.58" y2="144.78" width="0.1524" layer="91"/>
-<wire x1="68.58" y1="144.78" x2="60.96" y2="144.78" width="0.1524" layer="91"/>
-<wire x1="60.96" y1="144.78" x2="30.48" y2="144.78" width="0.1524" layer="91"/>
-<wire x1="30.48" y1="144.78" x2="25.4" y2="144.78" width="0.1524" layer="91"/>
-<wire x1="83.82" y1="144.78" x2="68.58" y2="144.78" width="0.1524" layer="91"/>
-<junction x="68.58" y="144.78"/>
-<wire x1="60.96" y1="76.2" x2="60.96" y2="144.78" width="0.1524" layer="91"/>
-<junction x="60.96" y="144.78"/>
-<pinref part="R2" gate="G$1" pin="2"/>
-<wire x1="30.48" y1="142.24" x2="30.48" y2="144.78" width="0.1524" layer="91"/>
-<junction x="30.48" y="144.78"/>
-<pinref part="X1" gate="-2" pin="KL"/>
+<wire x1="83.82" y1="144.78" x2="144.78" y2="144.78" width="0.1524" layer="91"/>
+<junction x="144.78" y="144.78"/>
+<pinref part="X2" gate="-2" pin="KL"/>
+<wire x1="30.48" y1="76.2" x2="60.96" y2="76.2" width="0.1524" layer="91"/>
 </segment>
 </net>
@@
 <segment>
 <pinref part="IC2" gate="G$1" pin="VBS"/>
-<wire x1="73.66" y1="149.86" x2="73.66" y2="111.76" width="0.1524" layer="91"/>
-<wire x1="73.66" y1="111.76" x2="40.64" y2="111.76" width="0.1524" layer="91"/>
-<pinref part="D1" gate="1" pin="A"/>
-<wire x1="43.18" y1="93.98" x2="40.64" y2="93.98" width="0.1524" layer="91"/>
-<wire x1="40.64" y1="93.98" x2="40.64" y2="111.76" width="0.1524" layer="91"/>
-<junction x="40.64" y="111.76"/>
+<wire x1="73.66" y1="149.86" x2="73.66" y2="142.24" width="0.1524" layer="91"/>
+<wire x1="73.66" y1="142.24" x2="40.64" y2="142.24" width="0.1524" layer="91"/>
 <pinref part="X1" gate="-1" pin="KL"/>
-<wire x1="40.64" y1="111.76" x2="40.64" y2="157.48" width="0.1524" layer="91"/>
+<wire x1="40.64" y1="142.24" x2="40.64" y2="157.48" width="0.1524" layer="91"/>
 <wire x1="40.64" y1="157.48" x2="22.86" y2="157.48" width="0.1524" layer="91"/>
 </segment>
@@
 <wire x1="68.58" y1="53.34" x2="33.02" y2="53.34" width="0.1524" layer="91"/>
 <label x="35.56" y="53.34" size="1.778" layer="95"/>
-<pinref part="X1" gate="-4" pin="KL"/>
+<pinref part="X2" gate="-3" pin="KL"/>
 </segment>
 </net>
@@
 <wire x1="50.8" y1="48.26" x2="50.8" y2="50.8" width="0.1524" layer="91"/>
 <wire x1="33.02" y1="48.26" x2="50.8" y2="48.26" width="0.1524" layer="91"/>
-<pinref part="X1" gate="-5" pin="KL"/>
+<pinref part="X2" gate="-4" pin="KL"/>
 </segment>
 </net>
@@
 </segment>
 </net>
+<net name="N$5" class="0">
+<segment>
+<pinref part="X2" gate="-1" pin="KL"/>
+<pinref part="D1" gate="1" pin="A"/>
+<wire x1="30.48" y1="93.98" x2="43.18" y2="93.98" width="0.1524" layer="91"/>
+</segment>
+</net>
+<net name="N$9" class="0">
+<segment>
+<pinref part="IC2" gate="G$1" pin="IN+"/>
+<wire x1="68.58" y1="149.86" x2="68.58" y2="144.78" width="0.1524" layer="91"/>
+<wire x1="68.58" y1="144.78" x2="30.48" y2="144.78" width="0.1524" layer="91"/>
+<pinref part="R2" gate="G$1" pin="2"/>
+<wire x1="30.48" y1="142.24" x2="30.48" y2="144.78" width="0.1524" layer="91"/>
+<junction x="30.48" y="144.78"/>
+<wire x1="30.48" y1="144.78" x2="25.4" y2="144.78" width="0.1524" layer="91"/>
+<pinref part="X1" gate="-2" pin="KL"/>
+</segment>
+</net>

Commit message: revertet some changes
Connections:
- removed net N$5: D1.A, X2-1.KL
- removed net N$9: IC2.IN+, R2.2, X1-2.KL
- net 12V: now also D1.A
- net GND: now also IC2.IN+, R2.2, X1-2.KL; no longer X2-2.KL
Other:
- note removed: "Supply voltage for ESP32 from NEMA Bus"
Changed lines of the file:
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@@
 <text x="2.54" y="132.08" size="1.778" layer="97">To Load</text>
 <text x="2.54" y="160.02" size="1.778" layer="97">Battery +</text>
-<text x="165.1" y="33.02" size="1.778" layer="97">Supply voltage for ESP32 from NEMA Bus</text>
 <text x="255.016" y="5.842" size="5.08" layer="97">A</text>
 </plain>
@@
 <instance part="X1" gate="-3" x="20.32" y="129.54" smashed="yes">
 <attribute name="NAME" x="19.05" y="130.429" size="1.778" layer="95" rot="R180"/>
-</instance>
-<instance part="X2" gate="-1" x="25.4" y="93.98" smashed="yes">
-<attribute name="NAME" x="24.13" y="94.869" size="1.778" layer="95" rot="R180"/>
-</instance>
-<instance part="X2" gate="-2" x="25.4" y="76.2" smashed="yes">
-<attribute name="NAME" x="24.13" y="77.089" size="1.778" layer="95" rot="R180"/>
 </instance>
 <instance part="X2" gate="-3" x="27.94" y="53.34" smashed="yes">
@@
 <wire x1="83.82" y1="144.78" x2="144.78" y2="144.78" width="0.1524" layer="91"/>
 <junction x="144.78" y="144.78"/>
-<pinref part="X2" gate="-2" pin="KL"/>
-<wire x1="30.48" y1="76.2" x2="60.96" y2="76.2" width="0.1524" layer="91"/>
+<pinref part="IC2" gate="G$1" pin="IN+"/>
+<wire x1="68.58" y1="149.86" x2="68.58" y2="144.78" width="0.1524" layer="91"/>
+<wire x1="68.58" y1="144.78" x2="60.96" y2="144.78" width="0.1524" layer="91"/>
+<pinref part="R2" gate="G$1" pin="2"/>
+<wire x1="60.96" y1="144.78" x2="30.48" y2="144.78" width="0.1524" layer="91"/>
+<wire x1="30.48" y1="142.24" x2="30.48" y2="144.78" width="0.1524" layer="91"/>
+<junction x="30.48" y="144.78"/>
+<wire x1="30.48" y1="144.78" x2="25.4" y2="144.78" width="0.1524" layer="91"/>
+<pinref part="X1" gate="-2" pin="KL"/>
+<wire x1="60.96" y1="76.2" x2="60.96" y2="144.78" width="0.1524" layer="91"/>
+<junction x="60.96" y="144.78"/>
 </segment>
 </net>
@@
 <segment>
 <pinref part="IC2" gate="G$1" pin="VBS"/>
-<wire x1="73.66" y1="149.86" x2="73.66" y2="142.24" width="0.1524" layer="91"/>
-<wire x1="73.66" y1="142.24" x2="40.64" y2="142.24" width="0.1524" layer="91"/>
+<wire x1="73.66" y1="149.86" x2="73.66" y2="124.46" width="0.1524" layer="91"/>
+<wire x1="73.66" y1="124.46" x2="40.64" y2="124.46" width="0.1524" layer="91"/>
 <pinref part="X1" gate="-1" pin="KL"/>
-<wire x1="40.64" y1="142.24" x2="40.64" y2="157.48" width="0.1524" layer="91"/>
+<wire x1="40.64" y1="124.46" x2="40.64" y2="157.48" width="0.1524" layer="91"/>
 <wire x1="40.64" y1="157.48" x2="22.86" y2="157.48" width="0.1524" layer="91"/>
+<pinref part="D1" gate="1" pin="A"/>
+<wire x1="43.18" y1="93.98" x2="40.64" y2="93.98" width="0.1524" layer="91"/>
+<wire x1="40.64" y1="93.98" x2="40.64" y2="124.46" width="0.1524" layer="91"/>
+<junction x="40.64" y="124.46"/>
 </segment>
 </net>
@@
 </segment>
 </net>
-<net name="N$5" class="0">
-<segment>
-<pinref part="X2" gate="-1" pin="KL"/>
-<pinref part="D1" gate="1" pin="A"/>
-<wire x1="30.48" y1="93.98" x2="43.18" y2="93.98" width="0.1524" layer="91"/>
-</segment>
-</net>
-<net name="N$9" class="0">
-<segment>
-<pinref part="IC2" gate="G$1" pin="IN+"/>
-<wire x1="68.58" y1="149.86" x2="68.58" y2="144.78" width="0.1524" layer="91"/>
-<wire x1="68.58" y1="144.78" x2="30.48" y2="144.78" width="0.1524" layer="91"/>
-<pinref part="R2" gate="G$1" pin="2"/>
-<wire x1="30.48" y1="142.24" x2="30.48" y2="144.78" width="0.1524" layer="91"/>
-<junction x="30.48" y="144.78"/>
-<wire x1="30.48" y1="144.78" x2="25.4" y2="144.78" width="0.1524" layer="91"/>
-<pinref part="X1" gate="-2" pin="KL"/>
-</segment>
-</net>

Commit message: added some missing values
Parts:
- IC1: value 5V -> R-78E05-1.0
Changed lines of the file:
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@@
 <parts>
 <part name="ESP1" library="_esp32" deviceset="ESP32-NODEMCU" device="" value="ESP32 NodeMCU"/>
-<part name="IC1" library="v-reg" library_urn="urn:adsk.eagle:library:409" deviceset="78XXS" device="" package3d_urn="urn:adsk.eagle:package:30342/1" value="5V"/>
+<part name="IC1" library="v-reg" library_urn="urn:adsk.eagle:library:409" deviceset="78XXS" device="" package3d_urn="urn:adsk.eagle:package:30342/1" value="R-78E05-1.0"/>
 <part name="IC3" library="_eigene" deviceset="MCP2562" device=""/>
 <part name="FRAME1" library="frames" library_urn="urn:adsk.eagle:library:229" deviceset="DINA4_L" device=""/>

Commit message: schema updated
Parts:
- ESP1: value ESP32 NodeMCU -> ESP32 CH340C Ultra Low Power Core Typ-C
Other:
- note added: "+12V und GND vom NMEA Bus dürfen nicht angeschlossen werden"
- moved on the sheet: X1-1
Changed lines of the file:
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@@
 </classes>
 <parts>
-<part name="ESP1" library="_esp32" deviceset="ESP32-NODEMCU" device="" value="ESP32 NodeMCU"/>
+<part name="ESP1" library="_esp32" deviceset="ESP32-NODEMCU" device="" value="ESP32 CH340C Ultra Low Power Core Typ-C"/>
 <part name="IC1" library="v-reg" library_urn="urn:adsk.eagle:library:409" deviceset="78XXS" device="" package3d_urn="urn:adsk.eagle:package:30342/1" value="R-78E05-1.0"/>
 <part name="IC3" library="_eigene" deviceset="MCP2562" device=""/>
@@
 <text x="5.08" y="48.26" size="1.778" layer="97">CANL = blau
 CANH = weiss</text>
-<text x="2.54" y="147.32" size="1.778" layer="97">Battery -</text>
-<text x="2.54" y="132.08" size="1.778" layer="97">To Load</text>
-<text x="2.54" y="160.02" size="1.778" layer="97">Battery +</text>
+<text x="11.684" y="145.542" size="1.778" layer="97" rot="R180">Battery -</text>
+<text x="11.938" y="130.302" size="1.778" layer="97" rot="R180">To Load</text>
+<text x="11.938" y="158.496" size="1.778" layer="97" rot="R180">Battery +</text>
 <text x="255.016" y="5.842" size="5.08" layer="97">A</text>
+<text x="8.382" y="77.724" size="1.778" layer="97">+12V und GND vom NMEA Bus
+dürfen nicht angeschlossen werden</text>
 </plain>
 <instances>
 <instance part="ESP1" gate="G$1" x="180.34" y="114.3" smashed="yes">
-<attribute name="VALUE" x="170.18" y="144.78" size="1.778" layer="96"/>
-<attribute name="NAME" x="170.18" y="147.32" size="1.778" layer="95"/>
+<attribute name="VALUE" x="167.64" y="83.82" size="1.778" layer="96"/>
+<attribute name="NAME" x="167.64" y="86.36" size="1.778" layer="95"/>
 </instance>
 <instance part="IC1" gate="1" x="78.74" y="93.98" smashed="yes">
@@
 </instance>
 <instance part="IC3" gate="G$1" x="81.28" y="68.58" smashed="yes" rot="R180">
-<attribute name="NAME" x="91.44" y="40.64" size="1.778" layer="95" rot="R180"/>
-<attribute name="VALUE" x="91.44" y="43.18" size="1.778" layer="96" rot="R180"/>
+<attribute name="NAME" x="73.66" y="43.18" size="1.778" layer="95"/>
+<attribute name="VALUE" x="73.66" y="40.64" size="1.778" layer="96"/>
 </instance>
 <instance part="FRAME1" gate="G$1" x="0" y="0" smashed="yes"/>
@@
 <attribute name="VALUE" x="48.26" y="91.6686" size="1.778" layer="96"/>
 </instance>
-<instance part="X1" gate="-1" x="17.78" y="157.48" smashed="yes">
-<attribute name="NAME" x="16.51" y="158.369" size="1.778" layer="95" rot="R180"/>
+<instance part="X1" gate="-1" x="20.32" y="157.48" smashed="yes">
+<attribute name="NAME" x="19.05" y="158.369" size="1.778" layer="95" rot="R180"/>
 </instance>
 <instance part="X1" gate="-2" x="20.32" y="144.78" smashed="yes">
@@
 <pinref part="X1" gate="-1" pin="KL"/>
 <wire x1="40.64" y1="124.46" x2="40.64" y2="157.48" width="0.1524" layer="91"/>
-<wire x1="40.64" y1="157.48" x2="22.86" y2="157.48" width="0.1524" layer="91"/>
+<wire x1="40.64" y1="157.48" x2="25.4" y2="157.48" width="0.1524" layer="91"/>
 <pinref part="D1" gate="1" pin="A"/>
 <wire x1="43.18" y1="93.98" x2="40.64" y2="93.98" width="0.1524" layer="91"/>
@@
 </segment>
 </net>
+<net name="N$5" class="0">
+<segment>
+<wire x1="5.08" y1="76.2" x2="48.26" y2="76.2" width="0.1524" layer="91"/>
+<wire x1="48.26" y1="76.2" x2="48.26" y2="83.82" width="0.1524" layer="91"/>
+<wire x1="48.26" y1="83.82" x2="5.08" y2="83.82" width="0.1524" layer="91"/>
+<wire x1="5.08" y1="83.82" x2="5.08" y2="76.2" width="0.1524" layer="91"/>
+</segment>
+</net>
